Commit message: Imported upstream version '0.5.4' of 'upstream'

File: cob_description/urdf/cob3_base/base.gazebo.xacro (robot description, xacro)
@@ -3,8 +3,6 @@
   <xacro:macro name="cob_wheel_gazebo" params="suffix parent">
     <gazebo reference="${parent}_${suffix}_wheel_link">
-      <mu1 value="100.0" />
-      <mu2 value="100.0" />
-      <kp  value="1000000.0" />
-      <kd  value="1.0" />
+      <gravity>true</gravity>
+      <self_collide>false</self_collide>
       <material value="IPA/LightGrey"/>
     </gazebo>
@@ -12,35 +10,42 @@
   <xacro:macro name="cob_caster_gazebo" params="suffix">
     <gazebo reference="${suffix}_caster_rotation_link">
+      <gravity>true</gravity>
+      <self_collide>false</self_collide>
       <material value="IPA/Metal"/>
     </gazebo>
   </xacro:macro>
   <xacro:macro name="base_gazebo" params="name">
-  <gazebo reference="${name}_link">
-    <selfCollide>true</selfCollide>
-    <sensor name='${name}_contact_sensor' type='contact'>
-      <contact>
-        <collision>${name}_link_geom</collision>
-      </contact>
-      <plugin name="${name}_gazebo_ros_bumper_controller" filename="libgazebo_ros_bumper.so">
+    <gazebo reference="${name}_link">
+      <gravity>true</gravity>
+      <self_collide>false</self_collide>
+      <material>IPA/LightGrey</material>
+<!-- FXM: the contact sensor currently does not work (the reason is within gazebo, NOT the bumper_plugin) -->
+<!--
+      <sensor name='${name}_contact_sensor' type='contact'>
+        <always_on>true</always_on>
+        <update_rate>100.0</update_rate>
+        <contact>
+          <collision>${name}_link_geom</collision>
+          <topic>${name}_bumper</topic>
+        </contact>
+        <plugin name="${name}_gazebo_ros_bumper_controller" filename="libgazebo_ros_bumper.so">
+          <frameName>world</frameName>
+          <bumperTopicName>${name}_bumper</bumperTopicName>
+        </plugin>
+      </sensor>
+-->
+    </gazebo>
+    <gazebo>
+      <plugin name="p3d_base_controller" filename="libgazebo_ros_p3d.so">
         <alwaysOn>true</alwaysOn>
         <updateRate>100.0</updateRate>
-        <bumperTopicName>${name}_bumper</bumperTopicName>
-		<frameName>world</frameName>
-		</plugin>
-    </sensor>
-    <material>IPA/LightGrey</material>
-  </gazebo>
-    <gazebo>
-    <plugin name="p3d_base_controller" filename="libgazebo_ros_p3d.so">
-      <alwaysOn>true</alwaysOn>
-      <updateRate>100.0</updateRate>
-      <bodyName>${name}_link</bodyName>
-      <topicName>${name}_pose_ground_truth</topicName>
-      <gaussianNoise>0.01</gaussianNoise>
-      <frameName>map</frameName>
-      <xyzOffsets>25.7 25.7 0</xyzOffsets> <!-- initialize odometry for fake localization-->
-      <rpyOffsets>0 0 0</rpyOffsets>
-    </plugin>
-    <canonicalBody>${name}_footprint</canonicalBody>
+        <bodyName>${name}_link</bodyName>
+        <topicName>${name}_pose_ground_truth</topicName>
+        <frameName>map</frameName>
+        <xyzOffsets>25.7 25.7 0</xyzOffsets> <!-- initialize odometry for fake localization-->
+        <rpyOffsets>0 0 0</rpyOffsets>
+        <gaussianNoise>0.01</gaussianNoise>
+      </plugin>
+      <canonicalBody>${name}_footprint</canonicalBody>
     </gazebo>
   </xacro:macro>

File: cob_description/urdf/cob4_base/base.gazebo.xacro (robot description, xacro)
@@ -12,35 +12,41 @@
   <xacro:macro name="cob_caster_gazebo" params="suffix">
     <gazebo reference="${suffix}_caster_rotation_link">
+      <gravity>true</gravity>
+      <self_collide>false</self_collide>
       <material value="IPA/Metal" />
     </gazebo>
   </xacro:macro>
   <xacro:macro name="base_gazebo" params="name">
-  <gazebo reference="${name}_link">
-    <selfCollide>true</selfCollide>
-    <sensor name='${name}_contact_sensor' type='contact'>
-      <contact>
-        <collision>${name}_link_geom</collision>
-      </contact>
-      <plugin name="${name}_gazebo_ros_bumper_controller" filename="libgazebo_ros_bumper.so">
+    <gazebo reference="${name}_link">
+      <gravity>true</gravity>
+      <self_collide>false</self_collide>
+<!-- FXM: the contact sensor currently does not work (the reason is within gazebo, NOT the bumper_plugin) -->
+<!--
+      <sensor name='${name}_contact_sensor' type='contact'>
+        <always_on>true</always_on>
+        <update_rate>100.0</update_rate>
+        <contact>
+          <collision>${name}_link_geom</collision>
+          <topic>${name}_bumper</topic>
+        </contact>
+        <plugin name="${name}_gazebo_ros_bumper_controller" filename="libgazebo_ros_bumper.so">
+          <frameName>world</frameName>
+          <bumperTopicName>${name}_bumper</bumperTopicName>
+        </plugin>
+      </sensor>
+-->
+    </gazebo>
+    <gazebo>
+      <plugin name="p3d_base_controller" filename="libgazebo_ros_p3d.so">
         <alwaysOn>true</alwaysOn>
         <updateRate>100.0</updateRate>
-        <frameName>world</frameName>
-        <bumperTopicName>${name}_bumper</bumperTopicName>
+        <bodyName>${name}_link</bodyName>
+        <topicName>${name}_pose_ground_truth</topicName>
+        <frameName>map</frameName>
+        <xyzOffsets>25.7 25.7 0</xyzOffsets> <!-- initialize odometry for fake localization-->
+        <rpyOffsets>0 0 0</rpyOffsets>
+        <gaussianNoise>0.01</gaussianNoise>
       </plugin>
-    </sensor>
-    <material>IPA/DarkGrey</material>
-  </gazebo>
-    <gazebo>
-    <plugin name="p3d_base_controller" filename="libgazebo_ros_p3d.so">
-      <alwaysOn>true</alwaysOn>
-      <updateRate>100.0</updateRate>
-      <bodyName>${name}_link</bodyName>
-      <topicName>${name}_pose_ground_truth</topicName>
-      <gaussianNoise>0.01</gaussianNoise>
-      <frameName>map</frameName>
-      <xyzOffsets>25.7 25.7 0</xyzOffsets> <!-- initialize odometry for fake localization-->
-      <rpyOffsets>0 0 0</rpyOffsets>
-    </plugin>
-    <canonicalBody>${name}_footprint</canonicalBody>
+      <canonicalBody>${name}_footprint</canonicalBody>
     </gazebo>
   </xacro:macro>

File: cob_description/urdf/cob4_base/base.urdf.xacro (robot description, xacro)
@@ -22,25 +22,5 @@
   <property name="base_collision_size_z" value="0.04" />
   <xacro:macro name="base" params="name">
-    <link name="base_footprint">
-      <inertial>
-        <mass value="1.0" />
-        <origin xyz="0 0 0" />
-        <inertia ixx="0.01" ixy="0.0" ixz="0.0"
-             iyy="0.01" iyz="0.0" izz="0.01" />
-        </inertial>
-        <visual>
-        <origin xyz="0 0 0" rpy="0 0 0" />
-        <geometry>
-          <box size="0.01 0.01 0.01" />
-        </geometry>
-        <material name="IPA/LightGrey" />
-        </visual>
-        <collision>
-        <origin xyz="0 0 0.1" rpy="0 0 0" />
-        <geometry>
-          <box size="0.001 0.001 0.001" />
-        </geometry>
-        </collision>
-    </link>
+    <link name="base_footprint"/>
     <joint name="base_footprint_joint" type="fixed">
       <origin xyz="0 0 0" rpy="0 0 0" />
@@ -56,15 +36,14 @@
       </inertial>
       <visual>
-        <origin xyz="0 0 0.05" rpy="0 0 3.14159" />
+        <origin xyz="0 0 0.0" rpy="0 0 0" />
         <geometry>
-          <mesh filename="package://cob_description/meshes/cob4_base/base_link.stl"/>
+          <mesh filename="package://cob_description/meshes/cob4_base/base.dae"/>
           <!--box size="0.01 0.01 0.01" /-->
         </geometry>
-        <material name="IPA/LightGrey"/>
       </visual>
       <collision>
-        <origin xyz="0 0 0.05" rpy="0 0 3.14159" />
+        <origin xyz="0 0 0.0" rpy="0 0 0" />
         <geometry>
-          <mesh filename="package://cob_description/meshes/cob4_base/base_link.stl"/>
+          <mesh filename="package://cob_description/meshes/cob4_base/base_collision.stl"/>
           <!--box size="0.01 0.01 0.01" /-->
         </geometry>
@@ -152,6 +131,5 @@
         <origin xyz="0 0 0" rpy="0 0 0" />
         <geometry>
-          <!--mesh filename="package://cob_description/meshes/cob4_base/caster.stl"/-->
-          <box size="0.01 0.01 0.01" />
+          <mesh filename="package://cob_description/meshes/cob4_base/caster.stl"/>
         </geometry>
         <material name="IPA/LightGrey" />

File: cob_description/urdf/cob4_head/head.urdf.xacro (robot description, xacro)
@@ -4,10 +4,10 @@
   <xacro:include filename="$(find cob_description)/urdf/cob4_head/head.transmission.xacro" />
   <xacro:macro name="head" params="parent name *origin">
-    <joint name="head_base_joint" type="fixed">
+    <joint name="${name}_base_joint" type="fixed">
       <insert_block name="origin" />
-      <child link="head_base_link" />
+      <child link="${name}_base_link" />
       <parent link="${parent}"/>
     </joint>
-    <link name="head_base_link">
+    <link name="${name}_base_link">
       <inertial>
         <origin xyz="0 0 0" rpy="0 0 0"/>
@@ -16,8 +16,8 @@
       </inertial>
     </link>
-    <joint name="head_1_joint" type="revolute">
+    <joint name="${name}_1_joint" type="revolute">
       <origin xyz="0 0 0.0305" rpy="0 0 0"/>
-      <child link="head_1_link" />
-      <parent link="head_base_link"/>
+      <child link="${name}_1_link" />
+      <parent link="${name}_base_link"/>
       <calibration rising="${head_1_ref}"/>
       <axis xyz="0 0 1" />
@@ -25,5 +25,5 @@
       <limit effort="100" lower="-6.2831" upper="6.2831" velocity="1.4"/>
     </joint>
-    <link name="head_1_link">
+    <link name="${name}_1_link">
       <inertial>
         <origin xyz="0 0 0" rpy="0 0 0"/>
@@ -32,8 +32,8 @@
       </inertial>
     </link>
-    <joint name="head_2_joint" type="revolute">
+    <joint name="${name}_2_joint" type="revolute">
       <origin xyz="0 -0.07725 -0.00439" rpy="-0.349 0 0" />
-      <child link="head_2_link" />
-      <parent link="head_1_link"/>
+      <child link="${name}_2_link" />
+      <parent link="${name}_1_link"/>
       <calibration rising="${head_2_ref}"/>
       <axis xyz="0 0 1" />
@@ -41,5 +41,5 @@
       <limit effort="100" lower="-6.2831" upper="6.2831" velocity="1.4"/>
     </joint>
-    <link name="head_2_link">
+    <link name="${name}_2_link">
       <inertial>
         <origin xyz="0 0 0" rpy="0 0 0"/>
@@ -48,8 +48,8 @@
       </inertial>
     </link>
-    <joint name="head_3_joint" type="revolute">
-      <origin xyz="0 0.08001 0.06809" rpy="0.349 0 0" />
-      <child link="head_3_link" />
-      <parent link="head_2_link"/>
+    <joint name="${name}_3_joint" type="revolute">
+      <origin xyz="0 0.04668 0.0976" rpy="0.349 0 0" />
+      <child link="${name}_3_link" />
+      <parent link="${name}_2_link"/>
       <calibration rising="${head_3_ref}"/>
       <axis xyz="0 0 1" />
@@ -57,25 +57,29 @@
       <limit effort="100" lower="-6.2831" upper="6.2831" velocity="1.4"/>
     </joint>
-    <link name="head_3_link">
+    <link name="${name}_3_link">
       <inertial>
-      <mass value="10" />
-      <origin xyz="0 0 0" />
-      <inertia ixx="5.652232699207" ixy="-0.009719934438" ixz="1.293988226423"
-           iyy="5.669473158652" iyz="-0.007379583694" izz="3.683196351726" />
+        <mass value="1" />
+        <origin xyz="0 0 0" />
+        <inertia ixx="0.01" ixy="0" ixz="0" iyy="0.01" iyz="0" izz="0.01" />
       </inertial>
       <visual>
-      <origin xyz="0 0 0" rpy="0 0 0" />
-      <geometry>
-        <mesh filename="package://cob_description/meshes/cob4_head/head_link.stl"/>
-      </geometry>
-      <material name="IPA/LightGrey"/>
+        <origin xyz="0 0 0" rpy="0 0 0" />
+        <geometry>
+          <mesh filename="package://cob_description/meshes/cob4_head/head_link.dae"/>
+        </geometry>
       </visual>
       <collision>
-      <origin xyz="0 0 0" rpy="0 0 0" />
-      <geometry>
-        <box size="0.001 0.001 0.001" />
-      </geometry>
+        <origin xyz="0 0 0" rpy="0 0 0" />
+        <geometry>
+          <mesh filename="package://cob_description/meshes/cob4_head/head_link.dae"/>
+        </geometry>
       </collision>
     </link>
+    <joint name="${name}_center_joint" type="fixed">
+      <origin xyz="0.0 0.0 -0.28247" rpy="0 0 0" />
+      <child link="${name}_center_link" />
+      <parent link="${name}_3_link"/>
+    </joint>
+    <link name="${name}_center_link"/>
   <!-- extensions -->
   <xacro:head_gazebo name="${name}" />

File: cob_description/urdf/cob4_torso/torso.urdf.xacro (robot description, xacro)
@@ -3,82 +3,94 @@
   <xacro:include filename="$(find cob_description)/urdf/cob4_torso/torso.gazebo.xacro" />
   <xacro:include filename="$(find cob_description)/urdf/cob4_torso/torso.transmission.xacro" />
+  <xacro:include filename="$(find cob_description)/urdf/sensors/softkinetic.urdf.xacro" />
+  <xacro:include filename="$(find cob_description)/urdf/sensors/kinect.urdf.xacro" />
   <xacro:macro name="torso" params="parent name *origin">
-    <joint name="torso_base_joint" type="fixed">
+    <joint name="${name}_base_joint" type="fixed">
       <insert_block name="origin" />
-      <child link="torso_base_link" />
+      <child link="${name}_base_link" />
       <parent link="${parent}"/>
     </joint>
-    <link name="torso_base_link">
-      <inertial>
-        <origin xyz="0 0 0" rpy="0 0 0"/>
-        <mass value="0.1"/>
-        <inertia ixx="0.01" ixy="0" ixz="0" iyy="0.01" iyz="0" izz="0.01" />
-      </inertial>
+    <link name="${name}_base_link">
+       <xacro:cylinder_inertial radius="0.300" length="0.046" mass="5.0">
+        <origin xyz="0 0 0" rpy="0 0 0" />
+      </xacro:cylinder_inertial>
     </link>
-    <joint name="torso_1_joint" type="revolute">
+    <joint name="${name}_1_joint" type="revolute">
       <origin xyz="0 0 0.04642" rpy="0 0 0"/>
-      <child link="torso_1_link" />
-      <parent link="torso_base_link"/>
+      <child link="${name}_1_link" />
+      <parent link="${name}_base_link"/>
       <calibration rising="${torso_1_ref}"/>
       <axis xyz="0 0 1" />
-      <dynamics damping="0.1" />
+      <dynamics damping="0.0" friction="0.0"/>
       <limit effort="100" lower="-6.2831" upper="6.2831" velocity="1.4"/>
     </joint>
-    <link name="torso_1_link">
-      <inertial>
-        <origin xyz="0 0 0" rpy="0 0 0"/>
-        <mass value="2"/>
-        <inertia ixx="0.01" ixy="0" ixz="0" iyy="0.01" iyz="0" izz="0.01" />
-      </inertial>
+    <link name="${name}_1_link">
+      <xacro:hollow_spherical_cap_inertial r="0.295" h="0.075" t="0.010" mass="6">
+          <!--origin xyz="0.006 0.010 0.110" rpy="0 0 0"/-->
+          <origin xyz="0 0 0" rpy="0 0 0"/>
+      </xacro:hollow_spherical_cap_inertial>
     </link>
-    <joint name="torso_2_joint" type="revolute">
+    <joint name="${name}_2_joint" type="revolute">
       <origin xyz="0 -0.14734 0.07547" rpy="-0.5236 0 0" />
-      <child link="torso_2_link" />
-      <parent link="torso_1_link"/>
+      <child link="${name}_2_link" />
+      <parent link="${name}_1_link"/>
       <calibration rising="${torso_2_ref}"/>
       <axis xyz="0 0 1" />
-      <dynamics damping="0.1" />
+      <dynamics damping="0.0" friction="0.0"/>
       <limit effort="100" lower="-6.2831" upper="6.2831" velocity="1.4"/>
     </joint>
-    <link name="torso_2_link">
-      <inertial>
-        <origin xyz="0 0 0" rpy="0 0 0"/>
-        <mass value="2"/>
-        <inertia ixx="0.01" ixy="0" ixz="0" iyy="0.01" iyz="0" izz="0.01" />
-      </inertial>
+    <link name="${name}_2_link">
+        <xacro:spherical_cap_inertial r="0.295" h="0.075" mass="19.5">
+            <origin xyz="0.034 0.102 0.092" rpy="0.5236 0 0"/>
+        </xacro:spherical_cap_inertial>
     </link>
-    <joint name="torso_3_joint" type="revolute">
-      <origin xyz="0 0.06223 0.15206" rpy="0.5236 0 0" />
-      <child link="torso_3_link" />
-      <parent link="torso_2_link"/>
+    <joint name="${name}_3_joint" type="revolute">
+      <origin xyz="0 0.09228 0.13477" rpy="0.5236 0 0" />
+      <child link="${name}_3_link" />
+      <parent link="${name}_2_link"/>
       <calibration rising="${torso_3_ref}"/>
       <axis xyz="0 0 1" />
-      <dynamics damping="0.1" />
+      <dynamics damping="0.0" friction="0.0"/>
       <limit effort="100" lower="-6.2831" upper="6.2831" velocity="1.4"/>
     </joint>
-    <link name="torso_3_link">
-      <inertial>
-        <mass value="10" />
-        <origin xyz="0 0 0" />
-      <inertia ixx="5.652232699207" ixy="-0.009719934438" ixz="1.293988226423"
-             iyy="5.669473158652" iyz="-0.007379583694" izz="3.683196351726" />
-      </inertial>
+    <link name="${name}_3_link">
+       <xacro:cylinder_inertial radius="0.250" length="0.610" mass="23.8">
+        <origin xyz="-0.028 0.005 0.233" rpy="0 0 0" />
+      </xacro:cylinder_inertial>
       <visual>
         <origin xyz="0 0 0" rpy="0 0 0" />
         <geometry>
-          <mesh filename="package://cob_description/meshes/cob4_torso/torso_link.stl"/>
+          <mesh filename="package://cob_description/meshes/cob4_torso/torso_link.dae"/>
         </geometry>
-        <material name="IPA/LightGrey"/>
       </visual>
       <collision>
         <origin xyz="0 0 0" rpy="0 0 0" />
         <geometry>
-          <box size="0.001 0.001 0.001" />
+          <mesh filename="package://cob_description/meshes/cob4_torso/torso_link.dae"/>
+          <!--box size="0.001 0.001 0.001" /-->
         </geometry>
       </collision>
     </link>
-  <!-- extensions -->
-  <xacro:torso_gazebo name="torso" />
-  <xacro:torso_transmission name="torso" />
+    <joint name="${name}_center_joint" type="fixed">
+      <origin xyz="0.0 0.0 0.18566" rpy="0 0 0" />
+      <child link="${name}_center_link" />
+      <parent link="${name}_3_link"/>
+    </joint>
+    <link name="${name}_center_link"/>
+    <!-- left camera -->
+    <xacro:cob_kinect_v0 name="${name}_cam3d_left" ros_topic="torso_cam3d_left" parent="${name}_3_link">
+      <origin xyz="${torso_cam3d_left_x} ${torso_cam3d_left_y} ${torso_cam3d_left_z}" rpy="${torso_cam3d_left_roll} ${torso_cam3d_left_pitch} ${torso_cam3d_left_yaw}" />
+    </xacro:cob_kinect_v0>
+    <!-- right camera -->
+    <xacro:cob_kinect_v0 name="${name}_cam3d_right" ros_topic="torso_cam3d_right" parent="${name}_3_link">
+      <origin xyz="${torso_cam3d_right_x} ${torso_cam3d_right_y} ${torso_cam3d_right_z}" rpy="${torso_cam3d_right_roll} ${torso_cam3d_right_pitch} ${torso_cam3d_right_yaw}" />
+    </xacro:cob_kinect_v0>
+    <!-- down camera -->
+    <xacro:softkinetic name="${name}_cam3d_down" ros_topic="torso_cam3d_down" parent="${name}_3_link">
+      <origin xyz="${torso_cam3d_down_x} ${torso_cam3d_down_y} ${torso_cam3d_down_z}" rpy="${torso_cam3d_down_roll} ${torso_cam3d_down_pitch} ${torso_cam3d_down_yaw}" />
+    </xacro:softkinetic>
+    <!-- extensions -->
+    <xacro:torso_gazebo name="torso" />
+    <xacro:torso_transmission name="torso" />
   </xacro:macro>
 </robot>

File: cob_description/urdf/sensors/kinect.gazebo.xacro (robot description, xacro)
@@ -1,47 +1,51 @@
 <?xml version="1.0"?>
 <root xmlns:xacro="http://www.ros.org/wiki/xacro">
-<xacro:macro name="cob_kinect_gazebo_v0" params="name ros_topic">
-  <gazebo reference="${name}_frame">
-  <sensor type="depth" name="${name}_frame_sensor">
-    <always_on>true</always_on>
-    <update_rate>20.0</update_rate>
-    <camera>
-      <horizontal_fov>${62.0*M_PI/180.0}</horizontal_fov>
-      <image>
-        <format>R8G8B8</format>
-        <width>640</width>
-        <height>480</height>
-      </image>
-      <clip>
-        <near>0.1</near>
-        <far>100</far>
-      </clip>
-    </camera>
-    <plugin name="${name}_controller" filename="libgazebo_ros_openni_kinect.so">
-      <alwaysOn>true</alwaysOn>
-      <updateRate>20.0</updateRate>
-      <cameraName>${ros_topic}</cameraName>
-      <frameName>${name}_link</frameName>
-      <imageTopicName>${ros_topic}/rgb/image_raw</imageTopicName>
-      <depthImageTopicName>${ros_topic}/depth/image_raw</depthImageTopicName>
-      <pointCloudTopicName>${ros_topic}/depth/points</pointCloudTopicName>
-      <cameraInfoTopicName>${ros_topic}/rgb/camera_info</cameraInfoTopicName>
-      <depthImageCameraInfoTopicName>${ros_topic}/depth/camera_info</depthImageCameraInfoTopicName>
-      <pointCloudCutoff>0.5</pointCloudCutoff>
-      <baseline>0.2</baseline>
-      <hackBaseline>0.0</hackBaseline>
-      <distortionK1>0.0</distortionK1>
-      <distortionK2>0.0</distortionK2>
-      <distortionK3>0.0</distortionK3>
-      <distortionT1>0.0</distortionT1>
-      <distortionT2>0.0</distortionT2>
-      <CxPrime>0.0</CxPrime>
-      <Cx>0.0</Cx>
-      <Cy>0.0</Cy>
-      <focalLength>0.0</focalLength>
-    </plugin>
-  </sensor>
-    <material>IPA/LightGrey</material>
-  </gazebo>
-</xacro:macro>
+  <xacro:macro name="cob_kinect_gazebo_v0" params="name ros_topic">
+    <gazebo reference="${name}_frame">
+      <sensor type="depth" name="${name}_frame_sensor">
+        <always_on>true</always_on>
+        <update_rate>20.0</update_rate>
+        <camera>
+          <horizontal_fov>${62.0*M_PI/180.0}</horizontal_fov>
+          <image>
+            <format>R8G8B8</format>
+            <width>640</width>
+            <height>480</height>
+          </image>
+          <clip>
+            <near>0.1</near>
+            <far>100</far>
+          </clip>
+          <noise>
+            <type>gaussian</type>
+            <mean>0.0</mean>
+            <stddev>0.0</stddev>
+          </noise>
+        </camera>
+        <plugin name="${name}_controller" filename="libgazebo_ros_openni_kinect.so">
+          <updateRate>20.0</updateRate>
+          <cameraName>${ros_topic}</cameraName>
+          <frameName>${name}_link</frameName>
+          <imageTopicName>rgb/image_raw</imageTopicName>
+          <depthImageTopicName>depth/image_raw</depthImageTopicName>
+          <pointCloudTopicName>depth_registered/points</pointCloudTopicName>
+          <cameraInfoTopicName>rgb/camera_info</cameraInfoTopicName>
+          <depthImageCameraInfoTopicName>depth_registered/camera_info</depthImageCameraInfoTopicName>
+          <pointCloudCutoff>0.5</pointCloudCutoff>
+          <baseline>0.2</baseline>
+          <hackBaseline>0.0</hackBaseline>
+          <distortionK1>0.0</distortionK1>
+          <distortionK2>0.0</distortionK2>
+          <distortionK3>0.0</distortionK3>
+          <distortionT1>0.0</distortionT1>
+          <distortionT2>0.0</distortionT2>
+          <CxPrime>0.0</CxPrime>
+          <Cx>0.0</Cx>
+          <Cy>0.0</Cy>
+          <focalLength>0.0</focalLength>
+        </plugin>
+      </sensor>
+      <material>IPA/LightGrey</material>
+    </gazebo>
+  </xacro:macro>
 </root>
