Commit message: Imported upstream version '0.5.4' of 'upstream'

File: cob_description/urdf/sensors/kinect.urdf.xacro (robot description, xacro)
@@ -9,13 +9,11 @@
     </joint>
     <link name="${name}_link">
-      <inertial>
-        <mass value="0.01" />
-        <origin xyz="0 0 0" rpy="0 0 0"/>
-        <inertia ixx="0.0001" ixy="0" ixz="0" iyy="0.0001" iyz="0" izz="0.0001" />
-      </inertial>
+      <xacro:box_inertial x="0.18" y="0.035" z="0.05" mass="0.3">
+        <origin xyz="0 0 0" rpy="0 0 0" />
+      </xacro:box_inertial>
       <visual>
         <origin xyz="0 0 -0.03" rpy="0 0 0" />
         <geometry>
-          <box size="0.06 0.02 0.02"/>
+          <box size="0.02 0.02 0.02"/>
         </geometry>
         <material name="IPA/LightGrey" />
@@ -24,5 +22,5 @@
         <origin xyz="0 0 -0.03" rpy="0 0 0" />
         <geometry>
-           <box size="0.06 0.02 0.02"/>
+           <box size="0.02 0.02 0.02"/>
         </geometry>
       </collision>

File: cob_description/urdf/sensors/sick_s300_laser.gazebo.xacro (robot description, xacro)
@@ -3,34 +3,34 @@
   <xacro:macro name="sick_s300_laser_gazebo_v0" params="name ros_topic update_rate min_angle max_angle">
     <gazebo reference="${name}_link">
-    <sensor name="${name}" type="ray">
-      <always_on>true</always_on>
-      <update_rate>${update_rate}</update_rate>
-      <pose>0 0 0 0 0 0</pose>
-      <visualize>false</visualize>
-      <ray>
-        <scan>
-          <horizontal>
-            <samples>541</samples>
-            <resolution>1.0</resolution>
-            <min_angle>${min_angle}</min_angle>
-            <max_angle>${max_angle}</max_angle>
-          </horizontal>
-        </scan>
-        <range>
-          <min>0.05</min>
-          <max>30.0</max>
-          <resolution>0.03</resolution>
-        </range>
-      </ray>
-      <plugin name="gazebo_ros_${name}_controller" filename="libgazebo_ros_laser.so">
-          <gaussianNoise>0.005</gaussianNoise>
-          <alwaysOn>true</alwaysOn>
-          <updateRate>${update_rate}</updateRate>
+      <sensor name="${name}" type="ray">
+        <always_on>true</always_on>
+        <update_rate>${update_rate}</update_rate>
+        <pose>0 0 0 0 0 0</pose>
+        <visualize>false</visualize>
+        <ray>
+          <scan>
+            <horizontal>
+              <samples>541</samples>
+              <resolution>1.0</resolution>
+              <min_angle>${min_angle}</min_angle>
+              <max_angle>${max_angle}</max_angle>
+            </horizontal>
+          </scan>
+          <range>
+            <min>0.05</min>
+            <max>30.0</max>
+            <resolution>0.03</resolution>
+          </range>
+          <noise>
+            <type>gaussian</type>
+            <mean>0.0</mean>
+            <stddev>0.005</stddev>
+          </noise>
+        </ray>
+        <plugin name="gazebo_ros_${name}_controller" filename="libgazebo_ros_laser.so">
           <topicName>${ros_topic}</topicName>
           <frameName>${name}_link</frameName>
-          <hokuyoMinIntensity>101.0</hokuyoMinIntensity>
-      </plugin>
-    </sensor>
-      <!--material value="IPA/LightGrey" /-->
+        </plugin>
+      </sensor>
     </gazebo>
   </xacro:macro>

File: raw_description/urdf/base_long/base.gazebo.xacro (robot description, xacro)
@@ -3,9 +3,5 @@
   <xacro:macro name="cob_wheel_gazebo" params="suffix parent">
     <gazebo reference="${parent}_${suffix}_wheel_link">
-      <mu1 value="100.0" />
-      <mu2 value="100.0" />
-      <kp  value="1000000.0" />
-      <kd  value="1.0" />
-      <!--material value="IPA/YellowRubber" /-->
+      <material value="IPA/LightGrey"/>
     </gazebo>
   </xacro:macro>
@@ -17,4 +13,6 @@
   <xacro:macro name="cob_batteries_gazebo" params="name">   <!-- added for raw model - fxmlc -->
     <gazebo reference="${name}_battery">
+      <gravity>true</gravity>
+      <self_collide>false</self_collide>
       <material value="Gazebo/Black" />
     </gazebo>
@@ -22,18 +20,21 @@
   <xacro:macro name="cob_base_gazebo" params="name">
     <gazebo reference="${name}_link">
-      <selfCollide>true</selfCollide>
+      <gravity>true</gravity>
+      <self_collide>false</self_collide>
+<!-- FXM: the contact sensor currently does not work (the reason is within gazebo, NOT the bumper_plugin) -->
+<!--
       <sensor name='${name}_contact_sensor' type='contact'>
+        <always_on>true</always_on>
+        <update_rate>100.0</update_rate>
         <contact>
           <collision>${name}_link_geom</collision>
+          <topic>${name}_bumper</topic>
         </contact>
         <plugin name="${name}_gazebo_ros_bumper_controller" filename="libgazebo_ros_bumper.so">
-          <alwaysOn>true</alwaysOn>
-          <updateRate>100.0</updateRate>
           <frameName>world</frameName>
           <bumperTopicName>${name}_bumper</bumperTopicName>
         </plugin>
       </sensor>
-      <!--material>Gazebo/Grey</material-->
-      <!--material value="IPA/Metal" /-->
+-->
     </gazebo>
     <gazebo>
@@ -43,8 +44,8 @@
         <bodyName>${name}_link</bodyName>
         <topicName>${name}_pose_ground_truth</topicName>
-        <gaussianNoise>0.01</gaussianNoise>
         <frameName>map</frameName>
         <xyzOffsets>25.7 25.7 0</xyzOffsets>  <!-- initialize odometry for fake localization-->
         <rpyOffsets>0 0 0</rpyOffsets>
+        <gaussianNoise>0.01</gaussianNoise>
       </plugin>
       <canonicalBody>${name}_footprint</canonicalBody>

File: raw_description/urdf/base_short/base.gazebo.xacro (robot description, xacro)
@@ -3,18 +3,16 @@
   <xacro:macro name="cob_wheel_gazebo" params="suffix parent">
     <gazebo reference="${parent}_${suffix}_wheel_link">
-      <mu1 value="100.0" />
-      <mu2 value="100.0" />
-      <kp  value="1000000.0" />
-      <kd  value="1.0" />
-      <!--material value="IPA/YellowRubber" /-->
+      <!--material value="IPA/LightGrey"/-->
     </gazebo>
   </xacro:macro>
   <xacro:macro name="cob_caster_gazebo" params="suffix">
     <gazebo reference="${suffix}_caster_rotation_link">
-      <material value="IPA/Metal" />
+      <!--material value="IPA/Metal" /-->
     </gazebo>
   </xacro:macro>
   <xacro:macro name="cob_batteries_gazebo" params="name">   <!-- added for raw model - fxmlc -->
     <gazebo reference="${name}_battery">
+      <gravity>true</gravity>
+      <self_collide>false</self_collide>
       <material value="Gazebo/Black" />
     </gazebo>
@@ -22,17 +20,21 @@
   <xacro:macro name="cob_base_gazebo" params="name">
     <gazebo reference="${name}_link">
-      <selfCollide>true</selfCollide>
+      <gravity>true</gravity>
+      <self_collide>false</self_collide>
+<!-- FXM: the contact sensor currently does not work (the reason is within gazebo, NOT the bumper_plugin) -->
+<!--
       <sensor name='${name}_contact_sensor' type='contact'>
+        <always_on>true</always_on>
+        <update_rate>100.0</update_rate>
         <contact>
           <collision>${name}_link_geom</collision>
+          <topic>${name}_bumper</topic>
         </contact>
         <plugin name="${name}_gazebo_ros_bumper_controller" filename="libgazebo_ros_bumper.so">
-          <alwaysOn>true</alwaysOn>
-          <updateRate>100.0</updateRate>
+          <frameName>world</frameName>
           <bumperTopicName>${name}_bumper</bumperTopicName>
         </plugin>
       </sensor>
-      <!--material>Gazebo/Grey</material-->
-      <!--material value="IPA/Metal" /-->
+-->
     </gazebo>
     <gazebo>
@@ -42,8 +44,8 @@
         <bodyName>${name}_link</bodyName>
         <topicName>${name}_pose_ground_truth</topicName>
-        <gaussianNoise>0.01</gaussianNoise>
         <frameName>map</frameName>
         <xyzOffsets>25.7 25.7 0</xyzOffsets>  <!-- initialize odometry for fake localization-->
         <rpyOffsets>0 0 0</rpyOffsets>
+        <gaussianNoise>0.01</gaussianNoise>
       </plugin>
       <canonicalBody>${name}_footprint</canonicalBody>
